File: Es. 9 Kikad - Prossimità e Temperatura/Es. 9 Kikad - Prossimità e Temperatura.sch (KiCad schematic (older format))
At the start: 16 parts, among them P1 Power, P2 Analog, P3 Digital, P4 Digital, P5 CONN_01X01, P6 CONN_01X01, P7 CONN_01X01, P8 CONN_01X01

Commit message: Update Schema elettrico Kikad
Parts:
- added R?: 10K ohm, symbol Device:R
- added SW?: SW_Push, symbol Switch:SW_Push
Connections:
- net +5V: now also SW?.2
- net 5(**): now also R?.2, SW?.1; no longer U?.2 (IO)
- net 6(**): now also U?.2 (IO)
- net GND: now also R?.1
Other:
- moved on the sheet: U?
Changed lines of the file:
@@
 	5950 4800 6300 4800
-Wire Wire Line
-	5950 4300 6300 4300
 Wire Wire Line
 	5950 4200 6300 4200
@@
 L Sensor:DHT11 U?
 U 1 1 5C80658A
-P 8550 4400
-F 0 "U?" H 8321 4446 50  0000 R CNN
-F 1 "DHT11" H 8321 4355 50  0000 R CNN
-F 2 "" H 8700 4650 50  0001 C CNN
-F 3 "http://akizukidenshi.com/download/ds/aosong/DHT11.pdf" H 8700 4650 50  0001 C CNN
-	1    8550 4400
+P 8750 4300
+F 0 "U?" H 8521 4346 50  0000 R CNN
+F 1 "DHT11" H 8521 4255 50  0000 R CNN
+F 2 "" H 8900 4550 50  0001 C CNN
+F 3 "http://akizukidenshi.com/download/ds/aosong/DHT11.pdf" H 8900 4550 50  0001 C CNN
+	1    8750 4300
 	-1   0    0    -1
 $EndComp
@@
 L power:GND #PWR?
 U 1 1 5C8066F6
-P 8650 4850
-F 0 "#PWR?" H 8650 4600 50  0001 C CNN
-F 1 "GND" H 8655 4677 50  0000 C CNN
-F 2 "" H 8650 4850 50  0001 C CNN
-F 3 "" H 8650 4850 50  0001 C CNN
-	1    8650 4850
-	1    0    0    -1
-$EndComp
-Wire Wire Line
-	8650 4700 8650 4850
+P 8850 4750
+F 0 "#PWR?" H 8850 4500 50  0001 C CNN
+F 1 "GND" H 8855 4577 50  0000 C CNN
+F 2 "" H 8850 4750 50  0001 C CNN
+F 3 "" H 8850 4750 50  0001 C CNN
+	1    8850 4750
+	1    0    0    -1
+$EndComp
+Wire Wire Line
+	8850 4600 8850 4750
 $Comp
 L power:+5V #PWR?
 U 1 1 5C807A47
-P 8650 3950
-F 0 "#PWR?" H 8650 3800 50  0001 C CNN
-F 1 "+5V" V 8650 4150 50  0000 C CNN
-F 2 "" H 8650 3950 50  0000 C CNN
-F 3 "" H 8650 3950 50  0000 C CNN
-	1    8650 3950
-	1    0    0    -1
-$EndComp
-Wire Wire Line
-	8650 3950 8650 4100
-Wire Wire Line
-	5950 4400 8250 4400
+P 8850 3850
+F 0 "#PWR?" H 8850 3700 50  0001 C CNN
+F 1 "+5V" V 8850 4050 50  0000 C CNN
+F 2 "" H 8850 3850 50  0000 C CNN
+F 3 "" H 8850 3850 50  0000 C CNN
+	1    8850 3850
+	1    0    0    -1
+$EndComp
+Wire Wire Line
+	8850 3850 8850 4000
 $Comp
 L Connector_Generic:Conn_01x04 HC_SR05
@@
 Wire Wire Line
 	5950 4000 7600 4000
+$Comp
+L Switch:SW_Push SW?
+U 1 1 5C80D764
+P 8850 5500
+F 0 "SW?" H 8850 5785 50  0000 C CNN
+F 1 "SW_Push" H 8850 5694 50  0000 C CNN
+F 2 "" H 8850 5700 50  0001 C CNN
+F 3 "" H 8850 5700 50  0001 C CNN
+	1    8850 5500
+	1    0    0    -1
+$EndComp
+Wire Wire Line
+	5950 4300 8450 4300
+Wire Wire Line
+	8400 4400 8400 5500
+Wire Wire Line
+	8400 5500 8550 5500
+Wire Wire Line
+	5950 4400 8400 4400
+$Comp
+L Device:R R?
+U 1 1 5C81308D
+P 8550 5900
+F 0 "R?" H 8480 5854 50  0000 R CNN
+F 1 "10K ohm" H 8480 5945 50  0000 R CNN
+F 2 "" V 8480 5900 50  0001 C CNN
+F 3 "~" H 8550 5900 50  0001 C CNN
+	1    8550 5900
+	-1   0    0    1
+$EndComp
+$Comp
+L power:GND #PWR?
+U 1 1 5C8130DB
+P 8550 6300
+F 0 "#PWR?" H 8550 6050 50  0001 C CNN
+F 1 "GND" H 8555 6127 50  0000 C CNN
+F 2 "" H 8550 6300 50  0001 C CNN
+F 3 "" H 8550 6300 50  0001 C CNN
+	1    8550 6300
+	1    0    0    -1
+$EndComp
+Wire Wire Line
+	8550 6050 8550 6300
+Wire Wire Line
+	8550 5750 8550 5500
+Connection ~ 8550 5500
+Wire Wire Line
+	8550 5500 8650 5500
+$Comp
+L power:+5V #PWR?
+U 1 1 5C8145E1
+P 9350 5400
+F 0 "#PWR?" H 9350 5250 50  0001 C CNN
+F 1 "+5V" V 9350 5600 50  0000 C CNN
+F 2 "" H 9350 5400 50  0000 C CNN
+F 3 "" H 9350 5400 50  0000 C CNN
+	1    9350 5400
+	1    0    0    -1
+$EndComp
+Wire Wire Line
+	9350 5400 9350 5500
+Wire Wire Line
+	9350 5500 9050 5500
 $EndSCHEMATC
